File: PowerModule/GateDrive.kicad_sch (KiCad schematic)
At the start: 6 parts, among them U1 IR2184SPBF

Commit message: update
Parts:
- C2: footprint Capacitor_THT:C_Rect_L11.0mm_W5.1mm_P10.00mm_MKT -> Capacitor_THT:C_Rect_L9.0mm_W5.1mm_P7.50mm_MKT
Changed lines of the file:
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@@
 			)
 		)
-		(property "Footprint" "Capacitor_THT:C_Rect_L11.0mm_W5.1mm_P10.00mm_MKT"
+		(property "Footprint" "Capacitor_THT:C_Rect_L9.0mm_W5.1mm_P7.50mm_MKT"
 			(at 100.0252 55.88 0)
 			(effects
