File: PowerModule/Phase.kicad_sch (KiCad schematic)
At the start: 20 parts, among them J9 Screw_Terminal_01x01, Q1 IRF1407, Q2 IRF1407

Commit message: update
Parts:
- added C29: 10nF, Capacitor_THT:C_Rect_L7.2mm_W3.5mm_P5.00mm_FKS2_FKP2_MKS2_MKP2, symbol Device:C
- C10, C11: footprint Capacitor_THT:C_Rect_L11.0mm_W5.1mm_P10.00mm_MKT -> Capacitor_THT:C_Rect_L7.2mm_W3.5mm_P5.00mm_FKS2_FKP2_MKS2_MKP2
- C12: footprint Capacitor_THT:C_Rect_L18.0mm_W7.0mm_P15.00mm_FKS3_FKP3 -> Capacitor_THT:C_Rect_L9.0mm_W5.1mm_P7.50mm_MKT
Connections:
- net GND: now also C29.2
- net VDCH: now also C29.1
Other:
- moved on the sheet: C13, C14
Changed lines of the file:
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@@
 	)
 	(junction
-		(at 162.56 76.2)
+		(at 173.99 76.2)
 		(diameter 0)
 		(color 0 0 0 0)
@@
 	)
 	(junction
-		(at 162.56 90.17)
+		(at 173.99 90.17)
 		(diameter 0)
 		(color 0 0 0 0)
@@
 	)
 	(junction
+		(at 165.1 116.84)
+		(diameter 0)
+		(color 0 0 0 0)
+	)
+	(junction
 		(at 156.21 49.53)
 		(diameter 0)
@@
 	)
 	(junction
+		(at 165.1 49.53)
+		(diameter 0)
+		(color 0 0 0 0)
+	)
+	(junction
 		(at 124.46 62.23)
 		(diameter 0)
@@
 	(wire
 		(pts
-			(xy 156.21 116.84) (xy 162.56 116.84)
+			(xy 156.21 116.84) (xy 165.1 116.84)
 		)
 		(stroke
@@
 	(wire
 		(pts
-			(xy 162.56 76.2) (xy 162.56 78.74)
-		)
-		(stroke
-			(width 0)
-			(type default)
-		)
-	)
-	(wire
-		(pts
-			(xy 170.18 76.2) (xy 162.56 76.2)
+			(xy 173.99 76.2) (xy 173.99 78.74)
+		)
+		(stroke
+			(width 0)
+			(type default)
+		)
+	)
+	(wire
+		(pts
+			(xy 181.61 76.2) (xy 173.99 76.2)
 		)
 		(stroke
@@
 	(wire
 		(pts
+			(xy 165.1 49.53) (xy 173.99 49.53)
+		)
+		(stroke
+			(width 0)
+			(type default)
+		)
+	)
+	(wire
+		(pts
 			(xy 116.84 62.23) (xy 124.46 62.23)
 		)
@@
 	(wire
 		(pts
-			(xy 156.21 49.53) (xy 162.56 49.53)
+			(xy 156.21 49.53) (xy 165.1 49.53)
 		)
 		(stroke
@@
 	(wire
 		(pts
-			(xy 170.18 86.36) (xy 170.18 90.17)
+			(xy 181.61 86.36) (xy 181.61 90.17)
 		)
 		(stroke
@@
 	(wire
 		(pts
-			(xy 170.18 90.17) (xy 162.56 90.17)
+			(xy 181.61 90.17) (xy 173.99 90.17)
 		)
 		(stroke
@@
 	(wire
 		(pts
+			(xy 165.1 86.36) (xy 165.1 116.84)
+		)
+		(stroke
+			(width 0)
+			(type default)
+		)
+	)
+	(wire
+		(pts
+			(xy 165.1 49.53) (xy 165.1 78.74)
+		)
+		(stroke
+			(width 0)
+			(type default)
+		)
+	)
+	(wire
+		(pts
 			(xy 132.08 49.53) (xy 132.08 57.15)
 		)
@@
 	(wire
 		(pts
-			(xy 162.56 90.17) (xy 162.56 116.84)
+			(xy 173.99 90.17) (xy 173.99 116.84)
 		)
 		(stroke
@@
 	(wire
 		(pts
-			(xy 170.18 76.2) (xy 170.18 78.74)
+			(xy 181.61 76.2) (xy 181.61 78.74)
 		)
 		(stroke
@@
 	(wire
 		(pts
-			(xy 162.56 86.36) (xy 162.56 90.17)
+			(xy 173.99 86.36) (xy 173.99 90.17)
 		)
 		(stroke
@@
 	(wire
 		(pts
-			(xy 162.56 76.2) (xy 162.56 49.53)
+			(xy 173.99 76.2) (xy 173.99 49.53)
 		)
 		(stroke
@@
 		(pts
 			(xy 132.08 86.36) (xy 132.08 95.25)
+		)
+		(stroke
+			(width 0)
+			(type default)
+		)
+	)
+	(wire
+		(pts
+			(xy 165.1 116.84) (xy 173.99 116.84)
 		)
 		(stroke
@@
 			)
 		)
-		(property "Footprint" "Capacitor_THT:C_Rect_L11.0mm_W5.1mm_P10.00mm_MKT"
+		(property "Footprint" "Capacitor_THT:C_Rect_L7.2mm_W3.5mm_P5.00mm_FKS2_FKP2_MKS2_MKP2"
 			(at 139.3952 62.23 0)
 			(effects
@@
 			)
 		)
-		(property "Footprint" "Capacitor_THT:C_Rect_L18.0mm_W7.0mm_P15.00mm_FKS3_FKP3"
+		(property "Footprint" "Capacitor_THT:C_Rect_L9.0mm_W5.1mm_P7.50mm_MKT"
 			(at 157.1752 86.36 0)
 			(effects
@@
 	(symbol
 		(lib_id "Device:C_Polarized")
-		(at 162.56 82.55 0)
+		(at 173.99 82.55 0)
 		(unit 1)
 		(exclude_from_sim no)
@@
 		(dnp no)
 		(property "Reference" "C13"
-			(at 164.338 78.74 0)
+			(at 175.768 78.74 0)
 			(effects
 				(font
@@
 		)
 		(property "Value" "220uF"
-			(at 160.782 85.09 0)
+			(at 172.212 85.09 0)
 			(effects
 				(font
@@
 		)
 		(property "Footprint" "LibMain:CP_Radial_Horizontal_P5.00_Up"
-			(at 163.5252 86.36 0)
+			(at 174.9552 86.36 0)
 			(effects
 				(font
@@
 		)
 		(property "Datasheet" "~"
-			(at 162.56 82.55 0)
+			(at 173.99 82.55 0)
 			(effects
 				(font
@@
 		)
 		(property "Description" "Polarized capacitor"
-			(at 162.56 82.55 0)
+			(at 173.99 82.55 0)
 			(effects
 				(font
@@
 			)
 		)
-		(property "Footprint" "Capacitor_THT:C_Rect_L11.0mm_W5.1mm_P10.00mm_MKT"
+		(property "Footprint" "Capacitor_THT:C_Rect_L7.2mm_W3.5mm_P5.00mm_FKS2_FKP2_MKS2_MKP2"
 			(at 139.3952 113.03 0)
 			(effects
@@
 	)
 	(symbol
+		(lib_id "Device:C")
+		(at 165.1 82.55 0)
+		(unit 1)
+		(exclude_from_sim no)
+		(in_bom yes)
+		(on_board yes)
+		(dnp no)
+		(fields_autoplaced yes)
+		(property "Reference" "C29"
+			(at 168.91 81.2799 0)
+			(effects
+				(font
+					(size 1.27 1.27)
+				)
+				(justify left)
+			)
+		)
+		(property "Value" "10nF"
+			(at 168.91 83.8199 0)
+			(effects
+				(font
+					(size 1.27 1.27)
+				)
+				(justify left)
+			)
+		)
+		(property "Footprint" "Capacitor_THT:C_Rect_L7.2mm_W3.5mm_P5.00mm_FKS2_FKP2_MKS2_MKP2"
+			(at 166.0652 86.36 0)
+			(effects
+				(font
+					(size 1.27 1.27)
+				)
+				(hide yes)
+			)
+		)
+		(property "Datasheet" "~"
+			(at 165.1 82.55 0)
+			(effects
+				(font
+					(size 1.27 1.27)
+				)
+				(hide yes)
+			)
+		)
+		(property "Description" "Unpolarized capacitor"
+			(at 165.1 82.55 0)
+			(effects
+				(font
+					(size 1.27 1.27)
+				)
+				(hide yes)
+			)
+		)
+		(pin "2"
+		)
+		(pin "1"
+		)
+		(instances
+			(project "PowerModule"
+				(path "/377d7bd9-5797-449c-aa80-62b80d7b56d8/14699ebe-f2d2-4155-aac0-4b159f9f7227"
+					(reference "C30")
+					(unit 1)
+				)
+				(path "/377d7bd9-5797-449c-aa80-62b80d7b56d8/4ca7d756-9094-484b-8a85-0e4c6bfcadf0"
+					(reference "C31")
+					(unit 1)
+				)
+				(path "/377d7bd9-5797-449c-aa80-62b80d7b56d8/8b6e91c1-c327-4148-83f9-0542a0b05d28"
+					(reference "C29")
+					(unit 1)
+				)
+			)
+		)
+	)
+	(symbol
 		(lib_id "Device:C_Polarized")
-		(at 170.18 82.55 0)
+		(at 181.61 82.55 0)
 		(unit 1)
 		(exclude_from_sim no)
@@
 		(dnp no)
 		(property "Reference" "C14"
-			(at 171.196 80.264 0)
+			(at 182.626 80.264 0)
 			(effects
 				(font
@@
 		)
 		(property "Value" "220uF"
-			(at 173.228 82.804 0)
+			(at 184.658 82.804 0)
 			(effects
 				(font
@@
 		)
 		(property "Footprint" "LibMain:CP_Radial_Horizontal_P5.00_Down"
-			(at 171.1452 86.36 0)
+			(at 182.5752 86.36 0)
 			(effects
 				(font
@@
 		)
 		(property "Datasheet" "~"
-			(at 170.18 82.55 0)
+			(at 181.61 82.55 0)
 			(effects
 				(font
@@
 		)
 		(property "Description" "Polarized capacitor"
-			(at 170.18 82.55 0)
-			(effects
-				(font
+			(at 181.61 82.55 0)
+			(effects
+				(font
