File: PowerModule/PowerModule.kicad_pcb (KiCad board)
At the start: 2 copper layers, 148.5 x 96.1 mm, 113 parts, among them J1 12V_IN, J10 Screw_Terminal_01x01, J11 Conn_01x01_Pin, J12 Conn_01x01_Pin, J13 Conn_01x01_Pin, J14 Conn_01x01_Pin, J15 Conn_01x01_Pin, J16 Conn_01x01_Pin, J17 Conn_01x01_Pin, J18 Conn_01x01_Pin, J19 Conn_01x01_Pin, J2 12V_IN, J20 Conn_01x01_Pin, J21 Conn_01x01_Pin, J22 Conn_01x01_Pin, J23 Screw_Terminal_01x01, J3 Conn_01x01_Pin, J4 Conn_01x01_Pin, J5 Screw_Terminal_01x01, J6 Screw_Terminal_01x01, J7 Conn_01x01_Pin, J8 Conn_01x01_Pin, J9 Screw_Terminal_01x01, Q1 IRF1407, Q2 IRF1407, Q3 IRF1407, Q4 IRF1407, Q5 IRF1407, Q6 IRF1407, U1 IR2184SPBF, U2 IR2184SPBF, U3 IR2184SPBF

Commit message: update
Parts:
- added C29: 10nF, Capacitor_THT:C_Rect_L7.2mm_W3.5mm_P5.00mm_FKS2_FKP2_MKS2_MKP2, F.Cu at (239.4, 38.6)
- added C30: 10nF, Capacitor_THT:C_Rect_L7.2mm_W3.5mm_P5.00mm_FKS2_FKP2_MKS2_MKP2, F.Cu at (140.9, 38.9)
- added C31: 10nF, Capacitor_THT:C_Rect_L7.2mm_W3.5mm_P5.00mm_FKS2_FKP2_MKS2_MKP2, F.Cu at (189.8, 38.7)
- C10, C11, C17, C18, C24, C25: footprint Capacitor_THT:C_Rect_L11.0mm_W5.1mm_P10.00mm_MKT -> Capacitor_THT:C_Rect_L7.2mm_W3.5mm_P5.00mm_FKS2_FKP2_MKS2_MKP2
- C12, C19, C26: footprint Capacitor_THT:C_Rect_L18.0mm_W7.0mm_P15.00mm_FKS3_FKP3 -> Capacitor_THT:C_Rect_L9.0mm_W5.1mm_P7.50mm_MKT
- C2, C4, C6: footprint Capacitor_THT:C_Rect_L11.0mm_W5.1mm_P10.00mm_MKT -> Capacitor_THT:C_Rect_L9.0mm_W5.1mm_P7.50mm_MKT
- moved C24 4.58 mm to (261.5, 32.6)
- moved C17 4.55 mm to (212.0, 32.6)
- moved C10 4.55 mm to (163.2, 32.6)
- moved C19 2.70 mm to (184.9, 38.4)
- moved C12 2.69 mm to (136.1, 38.5)
- moved C26 2.61 mm to (234.6, 38.3)
- moved R30 0.23 mm to (242.5, 42.7)
- moved R10 0.23 mm to (144.3, 43.0)
- moved R20 0.21 mm to (193.0, 43.0)
Routing:
- net /PhaseB: track 55.3 -> 52.2 mm
- net /PhaseC: track 57.7 -> 54.8 mm
- net /PhaseA: track 55.0 -> 52.1 mm
